Commit message: 阿克曼模式完善,解决雷达晃动问题,里程计错乱,tf树不完整等一系列问题

File: src/jzt_robot/urdf/jzt_mecanum copy.urdf (robot description, URDF)
Before this commit: robot jzAckermannRobot, 12 links, 11 joints
Links:
- removed link front_left_steer_link
- removed link front_right_steer_link
- removed link left_front_wheel_link
- removed link left_rear_wheel_link
- removed link right_front_wheel_link
- removed link right_rear_wheel_link
- added link front_left_wheel_link, mass 1.2; collision cylinder length=0.08 radius=0.108; visual box size=0.15 0.02 0.02
- added link front_right_wheel_link, mass 1.2; collision cylinder length=0.08 radius=0.108; visual box size=0.15 0.02 0.02
- added link rear_left_wheel_link, mass 1.2; collision cylinder length=0.08 radius=0.108; visual box size=0.15 0.02 0.02
- added link rear_right_wheel_link, mass 1.2; collision cylinder length=0.08 radius=0.108; visual box size=0.15 0.02 0.02
- link base_link: geometry collision box size=1.1 0.56 0.28; visual box size=1.1 0.56 0.28
- link camera_link: geometry collision box size=0.03 0.12 0.03; visual box size=0.03 0.12 0.03
Joints:
- removed joint front_left_steer_joint
- removed joint front_right_steer_joint
- removed joint left_front_wheel_joint
- removed joint left_rear_wheel_joint
- removed joint right_front_wheel_joint
- removed joint right_rear_wheel_joint
- added joint front_left_wheel_joint: type continuous, parent base_link, child front_left_wheel_link, origin xyz=0.40 0.28 0 rpy=0 0 0, axis 0 1 0
- added joint front_right_wheel_joint: type continuous, parent base_link, child front_right_wheel_link, origin xyz=0.40 -0.28 0 rpy=0 0 0, axis 0 1 0
- added joint rear_left_wheel_joint: type continuous, parent base_link, child rear_left_wheel_link, origin xyz=-0.40 0.28 0 rpy=0 0 0, axis 0 1 0
- added joint rear_right_wheel_joint: type continuous, parent base_link, child rear_right_wheel_link, origin xyz=-0.40 -0.28 0 rpy=0 0 0, axis 0 1 0
- joint base_joint: origin xyz=0.0 0.0 0.12 rpy=0 0 0 -> xyz=0.0 0.0 0.108 rpy=0 0 0
- joint camera_joint: origin xyz=0.56 0 0.25 rpy=0 0 0 -> xyz=0.536 0 0.14 rpy=0 0 0
- joint camera_optical_joint: origin xyz=0.06 0 0 rpy=-1.570796 0 -1.570796 -> xyz=0.015 0 0 rpy=-1.570796 0 -1.570796
- joint imu_joint: origin xyz=0 0 0 rpy=0 0 0 -> xyz=0 0 0.14 rpy=0 0 0
- joint laser_joint: origin xyz=0.40 0 0.36 rpy=0 0 0 -> xyz=0.40 0 0.32 rpy=0 0 0

File: src/jzt_robot/urdf/jzt_mecanum.urdf (robot description, URDF)
Before this commit: robot jzAckermannRobot, 12 links, 11 joints
Links:
- removed link front_left_steer_link
- removed link front_right_steer_link
- removed link left_front_wheel_link
- removed link left_rear_wheel_link
- removed link right_front_wheel_link
- removed link right_rear_wheel_link
- added link front_left_wheel_link, mass 1.2; collision cylinder length=0.08 radius=0.108; visual box size=0.15 0.02 0.02
- added link front_right_wheel_link, mass 1.2; collision cylinder length=0.08 radius=0.108; visual box size=0.15 0.02 0.02
- added link rear_left_wheel_link, mass 1.2; collision cylinder length=0.08 radius=0.108; visual box size=0.15 0.02 0.02
- added link rear_right_wheel_link, mass 1.2; collision cylinder length=0.08 radius=0.108; visual box size=0.15 0.02 0.02
- link base_link: geometry collision box size=1.1 0.56 0.28; visual box size=1.1 0.56 0.28
- link camera_link: geometry collision box size=0.03 0.12 0.03; visual box size=0.03 0.12 0.03
Joints:
- removed joint front_left_steer_joint
- removed joint front_right_steer_joint
- removed joint left_front_wheel_joint
- removed joint left_rear_wheel_joint
- removed joint right_front_wheel_joint
- removed joint right_rear_wheel_joint
- added joint front_left_wheel_joint: type continuous, parent base_link, child front_left_wheel_link, origin xyz=0.40 0.28 0 rpy=0 0 0, axis 0 1 0
- added joint front_right_wheel_joint: type continuous, parent base_link, child front_right_wheel_link, origin xyz=0.40 -0.28 0 rpy=0 0 0, axis 0 1 0
- added joint rear_left_wheel_joint: type continuous, parent base_link, child rear_left_wheel_link, origin xyz=-0.40 0.28 0 rpy=0 0 0, axis 0 1 0
- added joint rear_right_wheel_joint: type continuous, parent base_link, child rear_right_wheel_link, origin xyz=-0.40 -0.28 0 rpy=0 0 0, axis 0 1 0
- joint base_joint: origin xyz=0.0 0.0 0.12 rpy=0 0 0 -> xyz=0.0 0.0 0.108 rpy=0 0 0
- joint camera_joint: origin xyz=0.56 0 0.25 rpy=0 0 0 -> xyz=0.536 0 0.14 rpy=0 0 0
- joint camera_optical_joint: origin xyz=0.06 0 0 rpy=-1.570796 0 -1.570796 -> xyz=0.015 0 0 rpy=-1.570796 0 -1.570796
- joint imu_joint: origin xyz=0 0 0 rpy=0 0 0 -> xyz=0 0 0.14 rpy=0 0 0
- joint laser_joint: origin xyz=0.40 0 0.36 rpy=0 0 0 -> xyz=0.40 0 0.32 rpy=0 0 0
