Commit message: 全向麦克纳母轮机器人创建

File: src/jzt_robot/urdf/jzt_diff.urdf (robot description, URDF)
Before this commit: robot jzDiffRobot, 10 links, 9 joints
Links:
- added link camera_link, mass 0.05; collision box size=0.03 0.12 0.03; visual box size=0.03 0.12 0.03
- added link camera_optical_link
Joints:
- added joint camera_joint: type fixed, parent base_link, child camera_link, origin xyz=0.285 0 0.03 rpy=0 0 0
- added joint camera_optical_joint: type fixed, parent camera_link, child camera_optical_link, origin xyz=0.015 0 0 rpy=-1.570796 0 -1.570796

File: src/jzt_robot/urdf/mecanum/demo.urdf (robot description, URDF)
Before this commit: robot jzMecanumRobot, 10 links, 9 joints
Joints:
- joint base_joint: origin xyz=0.0 0.0 0.108 rpy=0 0 0 -> xyz=0 0 0.108 rpy=0 0 0
- joint camera_optical_joint: origin xyz=0.015 0 0 rpy=-1.570796 0 -1.570796 -> xyz=0.015 0 0 rpy=-1.570796327 0 -1.570796327
- joint front_left_wheel_joint: origin xyz=0.40 0.28 0 rpy=0 0 0 -> xyz=0.4 0.28 0.0 rpy=0 0 0
- joint front_right_wheel_joint: origin xyz=0.40 -0.28 0 rpy=0 0 0 -> xyz=0.4 -0.28 0.0 rpy=0 0 0
- joint rear_left_wheel_joint: origin xyz=-0.40 0.28 0 rpy=0 0 0 -> xyz=-0.4 0.28 0.0 rpy=0 0 0
- joint rear_right_wheel_joint: origin xyz=-0.40 -0.28 0 rpy=0 0 0 -> xyz=-0.4 -0.28 0.0 rpy=0 0 0
