Commit message: 跟踪算法演示

File: src/jzt_robot/urdf/mecanum/mecanum_base.xacro (robot description, xacro)
@@ -15,5 +15,5 @@
                 <box size="${base_box_x} ${base_box_y} ${base_box_z}" />
             </geometry>
-            <material name="white" />
+            <material name="light_red" />
         </visual>
         <collision>

File: src/jzt_robot/urdf/mecanum/mecanum_wheels.xacro (robot description, xacro)
@@ -26,5 +26,5 @@
                 </geometry>
             </collision>
-            0 <inertial>
+            <inertial>
                 <origin xyz="0 0 0" rpy="0 0 0" />
                 <mass value="${wheel_mass}" />
