Commit message: 双雷达机器人仿真+标定

File: src/jzt_robot/urdf/mecanum/common_properties.xacro (robot description, xacro)
@@ -8,5 +8,5 @@
     <xacro:property name="base_box_y" value="0.56" />
     <xacro:property name="base_box_z" value="0.216" />
-    <xacro:property name="base_mass" value="1.5" />
+    <xacro:property name="base_mass" value="30" />
     <!-- 底盘在 base_footprint 上的偏移，你的原值是 z=0.108 -->
     <xacro:property name="base_offset_z" value="0.108" />

File: src/jzt_robot/urdf/mecanum/ros2_control_sim.xacro (robot description, xacro)
@@ -30,5 +30,5 @@
     <gazebo>
         <plugin name="gazebo_ros2_control" filename="libgazebo_ros2_control.so">
-            <parameters>$(find jzt_robot)/config/mecanum_controllers.yaml</parameters>
+            <parameters>$(find jzt_robot)/config/ackermann_controllers.yaml</parameters>
         </plugin>
     </gazebo>
